File: hw/prototype/prototype.kicad_sch (KiCad schematic)
At the start: 26 parts, among them U1 TLC2274A

Commit message: Comments, fixed feedback resistor
Parts:
- R12, R6, R7: value 180K -> 150K
Connections:
- net GND: no longer C5.2, R1.1, R2.1, R3.1, R5.1, U1.4 (V+)
- new net VCC: C5.2, R1.1, R2.1, R3.1, R5.1, U1.4 (V+)
Changed lines of the file:
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@@
 	)
 	(junction
-		(at 149.86 73.66)
-		(diameter 0)
-		(color 0 0 0 0)
-	)
-	(junction
 		(at 247.65 130.81)
 		(diameter 0)
@@
 	(wire
 		(pts
-			(xy 151.13 73.66) (xy 149.86 73.66)
-		)
-		(stroke
-			(width 0)
-			(type default)
-		)
-	)
-	(wire
-		(pts
 			(xy 247.65 119.38) (xy 247.65 115.57)
 		)
@@
 	(wire
 		(pts
-			(xy 147.32 73.66) (xy 149.86 73.66)
+			(xy 147.32 73.66) (xy 151.13 73.66)
 		)
 		(stroke
@@
 	(wire
 		(pts
-			(xy 149.86 73.66) (xy 149.86 83.82)
-		)
-		(stroke
-			(width 0)
-			(type default)
-		)
-	)
-	(wire
-		(pts
 			(xy 172.72 129.54) (xy 172.72 130.81)
 		)
@@
 	(wire
 		(pts
-			(xy 137.16 83.82) (xy 149.86 83.82)
-		)
-		(stroke
-			(width 0)
-			(type default)
-		)
-	)
-	(wire
-		(pts
 			(xy 137.16 73.66) (xy 128.27 73.66)
 		)
@@
 			)
 		)
-		(property "Value" "180K"
+		(property "Value" "150K"
 			(at 227.33 46.99 90)
 			(show_name no)
@@
 			)
 		)
-		(property "Value" "180K"
+		(property "Value" "150K"
 			(at 151.13 102.87 90)
 			(show_name no)
@@
 			)
 		)
-		(property "Value" "180K"
+		(property "Value" "150K"
 			(at 151.13 46.99 90)
 			(show_name no)

Commit message: Added A4988 to schematic and datasheet to docs
Parts:
- added A1: Pololu_Breakout_A4988, Module:Pololu_Breakout-16_15.2x20.3mm, symbol Driver_Motor:Pololu_Breakout_A4988
- added C6: 100uF, PCM_Capacitor_THT_AKL:CP_Axial_L10.0mm_D4.5mm_P15.00mm_Horizontal, symbol Device:C
Connections:
- net GND: now also A1.1 (GND)
- net P0.04: no longer R13.2, R14.1
- net VCC: now also A1.2 (VDD); no longer R1.1, R2.1, R3.1
- new net: R13.2, R14.1
- new net: A1.13 (~{RESET}), A1.14 (~{SLEEP})
- new net +3V3: R1.1, R2.1, R3.1
- new net 1A: A1.4 (1A)
- new net 1B: A1.3 (1B)
- new net 2A: A1.5 (2A), A1.6 (2B)
- new net M_GND: A1.7 (GND), C6.2
- new net P1.03: A1.16 (DIR)
- new net P1.04: A1.15 (STEP)
- new net VMot: A1.8 (VMOT), C6.1
- no-connect marks 3 -> 7
Other:
- note added: "Stepper Motor Controller"
- moved on the sheet: C1, C2, C3, C4, C5, D4, D5, D6, R10, R11, R12, R13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

Commit message: Fixed errors in schematic, code testing in progress
Parts:
- removed C6: 100uF, PCM_Capacitor_THT_AKL:CP_Axial_L10.0mm_D4.5mm_P15.00mm_Horizontal, symbol Device:C
- added C7: 100uF, ECE445L:CP_Radial_Tantal200mil, symbol Project Library:C_Polarized
Connections:
- net +3V3 is gone; now on net VCC: R1.1, R2.1, R3.1
- net 2A: no longer A1.6 (2B)
- net GND: now also D4.2 (A), D5.2 (A), D6.2 (A); no longer D4.1 (K), D5.1 (K), D6.1 (K)
- net M_GND: now also C7.2
- net P0.03: now also R8.2, R9.1; no longer R10.2, R11.1
- net P0.28: now also R10.2, R11.1; no longer R8.2, R9.1
- net P0.29: now also U1.10 (+), U1.3 (+), U1.5 (+); no longer U1.2 (-), U1.6 (-), U1.9 (-)
- net VMot: now also C7.1
- net at C3.1, R7.1: now also D5.1 (K), U1.6 (-); no longer D5.2 (A), U1.5 (+)
- net at C4.1, R12.1: now also D6.1 (K), U1.9 (-); no longer D6.2 (A), U1.10 (+)
- net at C2.1, R6.1: now also D4.1 (K), U1.2 (-); no longer D4.2 (A), U1.3 (+)
- new net 2B: A1.6 (2B)
Other:
- moved on the sheet: D4, D5, D6

Commit message: Updated prototype schematic
Parts:
- removed C3, C4: 39pF, symbol Device:C
- removed D2, D3: LED_RED, LED_SMD:LED_Cree-XHP50_3V_HighDensity, symbol Device:LED
- removed D5, D6: D_Photo, OptoDevice:Kodenshi_LG206D, symbol Device:D_Photo
- removed R10, R13: 10k, symbol Device:R_US
- removed R11, R14: 15k, symbol Device:R_US
- removed R12, R7: 150K, symbol Device:R_US
- removed R2, R3: 330, symbol Device:R_US
- added U3: XIAO-ESP32-S3-DIP, Seeed_Studio_XIAO_Series:XIAO-ESP32-S3-DIP, symbol Seeed_Studio_XIAO_Series:XIAO-ESP32-S3-DIP
Connections:
- net GND: now also U3.13 (GND)
- net P0.03 renamed Vout_1
- net P0.29 renamed Vref
- net Vref: now also U3.3 (GPIO3_A2_D2); no longer U1.10 (+), U1.5 (+)
- net P1.03 renamed STEP
- net STEP: now also U3.2 (GPIO2_A1_D1)
- net P1.04 renamed DIR
- net DIR: now also U3.1 (GPIO1_A0_D0)
- new net V_USB: U3.14 (VBUS)
- new net Vin: U3.4 (GPIO4_A3_D3)
- no-connect marks 7 -> 21
Other:
- note removed: "LEDs"
- moved on the sheet: D1, R1
